File: kicad/nue-pcb.kicad_sch (KiCad schematic)
At the start: 160 parts, among them J1 Conn_01x04, J2 AVR-ISP-6, SW1 ESC, SW10 9, SW11 0, SW12 -, SW13 =, SW14 2U BACKSP, SW15 TAB150, SW16 Q, SW17 W, SW18 E, SW19 R, SW2 1, SW20 T, SW21 Y, SW22 U, SW23 I, SW24 O, SW25 P, SW26 CURL_L, SW27 CURL_R, SW28 1U RBKSP, SW29 CAPS, SW3 2, SW30 A, SW31 S, SW32 D, SW33 F, SW34 G, SW35 H, SW36 J, SW37 K, SW38 L, SW39 ;, SW4 3, SW40 ', SW41 PIPE150, SW42 ENTER_ANSI, SW43 LSHIFT225, SW44 ISO_PIPE, SW45 Z, SW46 X, SW47 C, SW48 V, SW49 B, SW5 4, SW50 N, SW51 M, SW52 <, SW53 >, SW54 ?, SW55 RSHIFT275, SW56 FN, SW57 LCTRL125, SW58 LWIN125, SW59 LALT125, SW6 5, SW60 SPACE625, SW61 RALT125, SW62 RWIN125, SW63 MENU, SW64 RCTRL125, SW65 1U LBACKSP, SW66 STEPPEDCAPS, SW67 ENTER_ISO, SW68 LSHIFT125, SW69 RSHIFT175, SW7 6, SW70 LCTRL150, SW71 LWIN100, SW72 LALT150, SW73 SPACE700, SW74 RALT150, SW75 RWIN100, SW76 RCTRL150, SW77 PIPE100, SW8 7, SW9 8, U1 ATmega32U4-MU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

Commit message: intial marker for caps_led in schematics
Parts:
- U: renamed from SW1; value ESC -> (none); footprint kestralib:MX100 -> (none)
- U: renamed from D1; value 1N4148 -> (none); footprint Diode_SMD:D_SOD-123 -> (none)
- U: renamed from D2; value 1N4148 -> (none); footprint Diode_SMD:D_SOD-123 -> (none)
- U: renamed from SW2; value 1 -> (none); footprint kestralib:MX100 -> (none)
- U: renamed from D3; value 1N4148 -> (none); footprint Diode_SMD:D_SOD-123 -> (none)
- U: renamed from SW3; value 2 -> (none); footprint kestralib:MX100 -> (none)
- U: renamed from D4; value 1N4148 -> (none); footprint Diode_SMD:D_SOD-123 -> (none)
- U: renamed from SW4; value 3 -> (none); footprint kestralib:MX100 -> (none)
- U: renamed from D5; value 1N4148 -> (none); footprint Diode_SMD:D_SOD-123 -> (none)
- U: renamed from SW5; value 4 -> (none); footprint kestralib:MX100 -> (none)
- U: renamed from D6; value 1N4148 -> (none); footprint Diode_SMD:D_SOD-123 -> (none)
- U: renamed from SW6; value 5 -> (none); footprint kestralib:MX100 -> (none)
- U: renamed from D7; value 1N4148 -> (none); footprint Diode_SMD:D_SOD-123 -> (none)
- U: renamed from SW7; value 6 -> (none); footprint kestralib:MX100 -> (none)
- U: renamed from D8; value 1N4148 -> (none); footprint Diode_SMD:D_SOD-123 -> (none)
- U: renamed from SW8; value 7 -> (none); footprint kestralib:MX100 -> (none)
- U: renamed from D9; value 1N4148 -> (none); footprint Diode_SMD:D_SOD-123 -> (none)
- U: renamed from SW9; value 8 -> (none); footprint kestralib:MX100 -> (none)
- U: renamed from D10; value 1N4148 -> (none); footprint Diode_SMD:D_SOD-123 -> (none)
- U: renamed from SW10; value 9 -> (none); footprint kestralib:MX100 -> (none)
- U: renamed from D11; value 1N4148 -> (none); footprint Diode_SMD:D_SOD-123 -> (none)
- U: renamed from SW11; value 0 -> (none); footprint kestralib:MX100 -> (none)
- U: renamed from D12; value 1N4148 -> (none); footprint Diode_SMD:D_SOD-123 -> (none)
- U: renamed from SW12; value - -> (none); footprint kestralib:MX100 -> (none)
- U: renamed from D13; value 1N4148 -> (none); footprint Diode_SMD:D_SOD-123 -> (none)
- U: renamed from SW13; value = -> (none); footprint kestralib:MX100 -> (none)
- U: renamed from D14; value 1N4148 -> (none); footprint Diode_SMD:D_SOD-123 -> (none)
- U: renamed from SW67; value ENTER_ISO -> (none); footprint kestralib:MXISOEnter -> (none)
- U: renamed from SW68; value LSHIFT125 -> (none); footprint kestralib:MX125 -> (none)
- U: renamed from SW70; value LCTRL150 -> (none); footprint kestralib:MX150 -> (none)
- U: renamed from SW15; value TAB150 -> (none); footprint kestralib:MX150 -> (none)
- U: renamed from SW16; value Q -> (none); footprint kestralib:MX100 -> (none)
- U: renamed from SW17; value W -> (none); footprint kestralib:MX100 -> (none)
- U: renamed from SW18; value E -> (none); footprint kestralib:MX100 -> (none)
- U: renamed from SW19; value R -> (none); footprint kestralib:MX100 -> (none)
- U: renamed from SW20; value T -> (none); footprint kestralib:MX100 -> (none)
- U: renamed from SW21; value Y -> (none); footprint kestralib:MX100 -> (none)
- U: renamed from SW22; value U -> (none); footprint kestralib:MX100 -> (none)
- U: renamed from SW23; value I -> (none); footprint kestralib:MX100 -> (none)
- U: renamed from SW24; value O -> (none); footprint kestralib:MX100 -> (none)
- U: renamed from SW25; value P -> (none); footprint kestralib:MX100 -> (none)
- U: renamed from SW26; value CURL_L -> (none); footprint kestralib:MX100 -> (none)
- U: renamed from SW27; value CURL_R -> (none); footprint kestralib:MX100 -> (none)
- U: renamed from SW28; value 1U RBKSP -> (none); footprint kestralib:MX100 -> (none)
- U: renamed from SW71; value LWIN100 -> (none); footprint kestralib:MX100 -> (none)
- U: renamed from SW29; value CAPS -> (none); footprint kestralib:MX175 -> (none)
- U: renamed from SW30; value A -> (none); footprint kestralib:MX100 -> (none)
- U: renamed from SW31; value S -> (none); footprint kestralib:MX100 -> (none)
- U: renamed from SW32; value D -> (none); footprint kestralib:MX100 -> (none)
- U: renamed from SW33; value F -> (none); footprint kestralib:MX100 -> (none)
- U: renamed from SW34; value G -> (none); footprint kestralib:MX100 -> (none)
- U: renamed from SW35; value H -> (none); footprint kestralib:MX100 -> (none)
- U: renamed from SW36; value J -> (none); footprint kestralib:MX100 -> (none)
- U: renamed from SW37; value K -> (none); footprint kestralib:MX100 -> (none)
- U: renamed from SW38; value L -> (none); footprint kestralib:MX100 -> (none)
- U: renamed from SW39; value ; -> (none); footprint kestralib:MX100 -> (none)
- U: renamed from SW40; value ' -> (none); footprint kestralib:MX100 -> (none)
- U: renamed from SW41; value PIPE150 -> (none); footprint kestralib:MX150 -> (none)
- U: renamed from SW42; value ENTER_ANSI -> (none); footprint kestralib:MX225R -> (none)
- U: renamed from SW72; value LALT150 -> (none); footprint kestralib:MX150 -> (none)
- U: renamed from SW43; value LSHIFT225 -> (none); footprint kestralib:MX225 -> (none)
- U: renamed from SW44; value ISO_PIPE -> (none); footprint kestralib:MX100 -> (none)
- U: renamed from SW45; value Z -> (none); footprint kestralib:MX100 -> (none)
- U: renamed from SW46; value X -> (none); footprint kestralib:MX100 -> (none)
- U: renamed from SW47; value C -> (none); footprint kestralib:MX100 -> (none)
- U: renamed from SW48; value V -> (none); footprint kestralib:MX100 -> (none)
- U: renamed from SW49; value B -> (none); footprint kestralib:MX100 -> (none)
- U: renamed from SW50; value N -> (none); footprint kestralib:MX100 -> (none)
- U: renamed from SW51; value M -> (none); footprint kestralib:MX100 -> (none)
- U: renamed from SW52; value < -> (none); footprint kestralib:MX100 -> (none)
- U: renamed from SW53; value > -> (none); footprint kestralib:MX100 -> (none)
- U: renamed from SW54; value ? -> (none); footprint kestralib:MX100 -> (none)
- U: renamed from SW55; value RSHIFT275 -> (none); footprint kestralib:MX275 -> (none)
- U: renamed from SW56; value FN -> (none); footprint kestralib:MX100 -> (none)
- U: renamed from SW73; value SPACE700 -> (none); footprint kestralib:MX700R -> (none)
- U: renamed from SW57; value LCTRL125 -> (none); footprint kestralib:MX125 -> (none)
- U: renamed from SW58; value LWIN125 -> (none); footprint kestralib:MX125 -> (none)
- U: renamed from SW59; value LALT125 -> (none); footprint kestralib:MX125 -> (none)
- U: renamed from SW60; value SPACE625 -> (none); footprint kestralib:MX625R -> (none)
- U: renamed from SW61; value RALT125 -> (none); footprint kestralib:MX125 -> (none)
- U: renamed from SW62; value RWIN125 -> (none); footprint kestralib:MX125 -> (none)
- U: renamed from SW63; value MENU -> (none); footprint kestralib:MX125 -> (none)
- U: renamed from SW64; value RCTRL125 -> (none); footprint kestralib:MX125 -> (none)
- U: renamed from SW77; value PIPE100 -> (none); footprint kestralib:MX100 -> (none)
- U: renamed from SW76; value RCTRL150 -> (none); footprint kestralib:MX150 -> (none)
- U: renamed from SW69; value RSHIFT175 -> (none); footprint kestralib:MX175 -> (none)
- U: renamed from SW14; value 2U BACKSP -> (none); footprint kestralib:MX200 -> (none)
- U: renamed from SW65; value 1U LBACKSP -> (none); footprint kestralib:MX100 -> (none)
- U: renamed from SW66; value STEPPEDCAPS -> (none); footprint kestralib:MX125 -> (none)
- U: renamed from D15; value 1N4148 -> (none); footprint Diode_SMD:D_SOD-123 -> (none)
- U: renamed from D16; value 1N4148 -> (none); footprint Diode_SMD:D_SOD-123 -> (none)
- U: renamed from D17; value 1N4148 -> (none); footprint Diode_SMD:D_SOD-123 -> (none)
- U: renamed from D18; value 1N4148 -> (none); footprint Diode_SMD:D_SOD-123 -> (none)
- U: renamed from D19; value 1N4148 -> (none); footprint Diode_SMD:D_SOD-123 -> (none)
- U: renamed from D20; value 1N4148 -> (none); footprint Diode_SMD:D_SOD-123 -> (none)
- U: renamed from D21; value 1N4148 -> (none); footprint Diode_SMD:D_SOD-123 -> (none)
- U: renamed from D22; value 1N4148 -> (none); footprint Diode_SMD:D_SOD-123 -> (none)
- U: renamed from D23; value 1N4148 -> (none); footprint Diode_SMD:D_SOD-123 -> (none)
- U: renamed from D24; value 1N4148 -> (none); footprint Diode_SMD:D_SOD-123 -> (none)
- U: renamed from D25; value 1N4148 -> (none); footprint Diode_SMD:D_SOD-123 -> (none)
- U: renamed from D26; value 1N4148 -> (none); footprint Diode_SMD:D_SOD-123 -> (none)
- U: renamed from D27; value 1N4148 -> (none); footprint Diode_SMD:D_SOD-123 -> (none)
- U: renamed from D28; value 1N4148 -> (none); footprint Diode_SMD:D_SOD-123 -> (none)
- U: renamed from D29; value 1N4148 -> (none); footprint Diode_SMD:D_SOD-123 -> (none)
- U: renamed from D30; value 1N4148 -> (none); footprint Diode_SMD:D_SOD-123 -> (none)
- U: renamed from D31; value 1N4148 -> (none); footprint Diode_SMD:D_SOD-123 -> (none)
- U: renamed from D32; value 1N4148 -> (none); footprint Diode_SMD:D_SOD-123 -> (none)
- U: renamed from D33; value 1N4148 -> (none); footprint Diode_SMD:D_SOD-123 -> (none)
- U: renamed from D34; value 1N4148 -> (none); footprint Diode_SMD:D_SOD-123 -> (none)
- U: renamed from D35; value 1N4148 -> (none); footprint Diode_SMD:D_SOD-123 -> (none)
- U: renamed from D36; value 1N4148 -> (none); footprint Diode_SMD:D_SOD-123 -> (none)
- U: renamed from D37; value 1N4148 -> (none); footprint Diode_SMD:D_SOD-123 -> (none)
- U: renamed from D38; value 1N4148 -> (none); footprint Diode_SMD:D_SOD-123 -> (none)
- U: renamed from D39; value 1N4148 -> (none); footprint Diode_SMD:D_SOD-123 -> (none)
- U: renamed from D40; value 1N4148 -> (none); footprint Diode_SMD:D_SOD-123 -> (none)
- U: renamed from D41; value 1N4148 -> (none); footprint Diode_SMD:D_SOD-123 -> (none)
- U: renamed from D42; value 1N4148 -> (none); footprint Diode_SMD:D_SOD-123 -> (none)
- U: renamed from D43; value 1N4148 -> (none); footprint Diode_SMD:D_SOD-123 -> (none)
- U: renamed from D44; value 1N4148 -> (none); footprint Diode_SMD:D_SOD-123 -> (none)
- U: renamed from D45; value 1N4148 -> (none); footprint Diode_SMD:D_SOD-123 -> (none)
- U: renamed from D46; value 1N4148 -> (none); footprint Diode_SMD:D_SOD-123 -> (none)
- U: renamed from D47; value 1N4148 -> (none); footprint Diode_SMD:D_SOD-123 -> (none)
- U: renamed from D48; value 1N4148 -> (none); footprint Diode_SMD:D_SOD-123 -> (none)
- U: renamed from D49; value 1N4148 -> (none); footprint Diode_SMD:D_SOD-123 -> (none)
- U: renamed from D50; value 1N4148 -> (none); footprint Diode_SMD:D_SOD-123 -> (none)
- U: renamed from D51; value 1N4148 -> (none); footprint Diode_SMD:D_SOD-123 -> (none)
- U: renamed from D52; value 1N4148 -> (none); footprint Diode_SMD:D_SOD-123 -> (none)
- U: renamed from D53; value 1N4148 -> (none); footprint Diode_SMD:D_SOD-123 -> (none)
- U: renamed from D54; value 1N4148 -> (none); footprint Diode_SMD:D_SOD-123 -> (none)
- U: renamed from D55; value 1N4148 -> (none); footprint Diode_SMD:D_SOD-123 -> (none)
- U: renamed from D56; value 1N4148 -> (none); footprint Diode_SMD:D_SOD-123 -> (none)
- U: renamed from D57; value 1N4148 -> (none); footprint Diode_SMD:D_SOD-123 -> (none)
- U: renamed from D58; value 1N4148 -> (none); footprint Diode_SMD:D_SOD-123 -> (none)
- U: renamed from D59; value 1N4148 -> (none); footprint Diode_SMD:D_SOD-123 -> (none)
- U: renamed from D60; value 1N4148 -> (none); footprint Diode_SMD:D_SOD-123 -> (none)
- U: renamed from D61; value 1N4148 -> (none); footprint Diode_SMD:D_SOD-123 -> (none)
- U: renamed from D62; value 1N4148 -> (none); footprint Diode_SMD:D_SOD-123 -> (none)
- U: renamed from D63; value 1N4148 -> (none); footprint Diode_SMD:D_SOD-123 -> (none)
- U: renamed from D64; value 1N4148 -> (none); footprint Diode_SMD:D_SOD-123 -> (none)
- U: renamed from U1; value ATmega32U4-MU -> (none); footprint Package_DFN_QFN:QFN-44-1EP_7x7mm_P0.5mm_EP5.2x5.2mm -> (none)
- U: renamed from SW74; value RALT150 -> (none); footprint kestralib:MX150 -> (none)
- U: renamed from SW75; value RWIN100 -> (none); footprint kestralib:MX100 -> (none)
- U: renamed from C1; value 1uF -> (none); footprint Capacitor_SMD:C_0603_1608Metric -> (none)
- U: renamed from C2; value 10uF -> (none); footprint Capacitor_SMD:C_0603_1608Metric -> (none)
- U: renamed from C3; value 0.1uF -> (none); footprint Capacitor_SMD:C_0603_1608Metric -> (none)
- U: renamed from C4; value 0.1uF -> (none); footprint Capacitor_SMD:C_0603_1608Metric -> (none)
- U: renamed from C5; value 0.1uF -> (none); footprint Capacitor_SMD:C_0603_1608Metric -> (none)
- U: renamed from J1; value Conn_01x04 -> (none); footprint kestralib:JST_BM04B-ASRS -> (none)
- U: renamed from SW_RST1; value SW_Push -> (none); footprint kestralib:pushbtn_C319436 -> (none)
- U: renamed from R3; value 22 -> (none); footprint Resistor_SMD:R_0603_1608Metric -> (none)
- U: renamed from R4; value 22 -> (none); footprint Resistor_SMD:R_0603_1608Metric -> (none)
- U: renamed from R1; value 10k -> (none); footprint Resistor_SMD:R_0603_1608Metric -> (none)
- U: renamed from Y1; value 16 MHz -> (none); footprint Crystal:Crystal_SMD_2520-4Pin_2.5x2.0mm -> (none)
- U: renamed from C6; value 22pF -> (none); footprint Capacitor_SMD:C_0603_1608Metric -> (none)
- U: renamed from C7; value 22pF -> (none); footprint Capacitor_SMD:C_0603_1608Metric -> (none)
- U: renamed from R2; value 1k -> (none); footprint Resistor_SMD:R_0603_1608Metric -> (none)
- U: renamed from J2; value AVR-ISP-6 -> (none); footprint kestralib:Conn_AVR_ISP_6 -> (none)
- U: renamed from H1; value StudioKestra Logo -> (none); footprint kestralib:sk-square-mask-md -> (none)
- U: renamed from H2; value Nue Logo -> (none); footprint kestralib:nue-logo -> (none)
- U: renamed from H3; value qmk-via logo -> (none); footprint kestralib:qmk-via -> (none)
Connections:
- net Caps_led: now reaches U.18 (PD0)
- no-connect marks 4 -> 3
